Commit message: feat: added map files

File: shreyas_bot/urdf/shreyas_bot.xacro (robot description, xacro)
@@ -2,4 +2,5 @@
 <robot name="shreyas_bot" xmlns:xacro="http://www.ros.org/wiki/xacro">
 <xacro:include filename="$(find shreyas_bot)/urdf/shreyas_bot.gazebo" />
+<xacro:include filename="$(find shreyas_bot)/urdf/shreyas_materials.xacro" />
   <link name="robot_footprint"></link>
   <joint name="robot_footprint_joint" type="fixed">
@@ -8,13 +9,14 @@
     <child link="chassis" />
   </joint>
+  <!-- chassis link -->
   <link name='chassis'>
     <pose>0 0 0.1 0 0 0</pose>
     <inertial>
-      <mass value="30.0"/>
+      <mass value="16.5"/>
       <origin xyz="0.0 0 0" rpy=" 0 0 0"/>
       <inertia
-          ixx="0.1" ixy="0" ixz="0"
-          iyy="0.1" iyz="0"
-          izz="0.1"
+          ixx="0.11" ixy="0" ixz="0"
+          iyy="0.11" iyz="0"
+          izz="0.11"
       />
     </inertial>
@@ -22,5 +24,5 @@
       <origin xyz="0 0 0" rpy=" 0 0 0"/>
       <geometry>
-        <box size=".8 .4 .2"/>
+        <box size=".44 .22 .11"/>
       </geometry>
     </collision>
@@ -28,11 +30,12 @@
       <origin xyz="0 0 0" rpy=" 0 0 0"/>
       <geometry>
-        <box size=".8 .4 .2"/>
-      </geometry>
+        <box size=".44 .22 .11"/>
+      </geometry>
+      <material name="blue"/>
     </visual>
     <collision name='back_caster_collision'>
-      <origin xyz="-0.30 0 -0.10" rpy=" 0 0 0"/>
-      <geometry>
-        <sphere radius="0.10"/>
+      <origin xyz="-0.165 0 -0.055" rpy=" 0 0 0"/>
+      <geometry>
+        <sphere radius="0.055"/>
       </geometry>
       <surface>
@@ -48,13 +51,13 @@
     </collision>
     <visual name='back_caster_visual'>
-      <origin xyz="-0.30 0 -0.10" rpy=" 0 0 0"/>
-      <geometry>
-        <sphere radius="0.10"/>
+      <origin xyz="-0.165 0 -0.055" rpy=" 0 0 0"/>
+      <geometry>
+        <sphere radius="0.055"/>
       </geometry>
     </visual>
     <collision name='front_caster_collision'>
-      <origin xyz="0.30 0 -0.10" rpy=" 0 0 0"/>
-      <geometry>
-        <sphere radius="0.10"/>
+      <origin xyz="0.165 0 -0.055" rpy=" 0 0 0"/>
+      <geometry>
+        <sphere radius="0.055"/>
       </geometry>
       <surface>
@@ -70,7 +73,7 @@
     </collision>
     <visual name='front_caster_visual'>
-      <origin xyz="0.30 0 -0.10" rpy=" 0 0 0"/>
-      <geometry>
-        <sphere radius="0.10"/>
+      <origin xyz="0.165 0 -0.055" rpy=" 0 0 0"/>
+      <geometry>
+        <sphere radius="0.055"/>
       </geometry>
     </visual>
@@ -80,10 +83,10 @@
     <pose>0 0 0 0 1.5707 1.5707</pose>
     <inertial>
-      <mass value="10.0"/>
+      <mass value="5.5"/>
       <origin xyz="0 0 0" rpy=" 0 1.5707 1.5707"/>
       <inertia
-          ixx="0.2" ixy="0" ixz="0"
-          iyy="0.2" iyz="0"
-          izz="0.2"
+          ixx="0.1" ixy="0" ixz="0"
+          iyy="0.1" iyz="0"
+          izz="0.1"
       />
     </inertial>
@@ -91,5 +94,5 @@
       <origin xyz="0 0 0" rpy=" 0 1.5707 1.5707"/>
       <geometry>
-        <cylinder length="0.10" radius="0.2"/>
+        <cylinder length="0.055" radius="0.11"/>
       </geometry>
     </collision>
@@ -97,5 +100,5 @@
       <origin xyz="0 0 0" rpy=" 0 1.5707 1.5707"/>
       <geometry>
-        <cylinder length="0.10" radius="0.2"/>
+        <cylinder length="0.055" radius="0.11"/>
       </geometry>
       <material name="green"/>
@@ -106,10 +109,10 @@
     <pose>0 0 0 0 -1.5707 1.5707</pose>
     <inertial>
-      <mass value="10.0"/>
+      <mass value="5.5"/>
       <origin xyz="0 0 0" rpy=" 0 -1.5707 1.5707"/>
       <inertia
-          ixx="0.2" ixy="0" ixz="0"
-          iyy="0.2" iyz="0"
-          izz="0.2"
+          ixx="0.1" ixy="0" ixz="0"
+          iyy="0.1" iyz="0"
+          izz="0.1"
       />
     </inertial>
@@ -117,5 +120,5 @@
       <origin xyz="0 0 0" rpy=" 0 -1.5707 1.5707"/>
       <geometry>
-        <cylinder length="0.10" radius="0.2"/>
+        <cylinder length="0.055" radius="0.11"/>
       </geometry>
     </collision>
@@ -123,5 +126,5 @@
       <origin xyz="0 0 0" rpy=" 0 -1.5707 1.5707"/>
       <geometry>
-        <cylinder length="0.10" radius="0.2"/>
+        <cylinder length="0.055" radius="0.11"/>
       </geometry>
       <material name="green"/>
@@ -181,23 +184,23 @@
   <!-- left wheel joint -->
   <joint type="continuous" name="left_wheel_hinge">
-    <origin xyz="0 0.30 0" rpy="0 0 0"/>
+    <origin xyz="0 0.165 0" rpy="0 0 0"/>
     <child link="left_wheel"/>
     <parent link="chassis"/>
     <axis xyz="0 1 0" rpy="0 0 0"/>
-    <limit effort="20000" velocity="2000"/>
-    <joint_properties damping="2.0" friction="2.0"/>
-  </joint>
-    <!-- right wheel joint -->
+    <limit effort="11000" velocity="1000"/>
+    <joint_properties damping="1.0" friction="1.0"/>
+  </joint>
+  <!-- right wheel joint -->
   <joint type="continuous" name="right_wheel_hinge">
-    <origin xyz="0 -0.30 0" rpy="0 0 0"/>
+    <origin xyz="0 -0.165 0" rpy="0 0 0"/>
     <child link="right_wheel"/>
     <parent link="chassis"/>
     <axis xyz="0 1 0" rpy="0 0 0"/>
-    <limit effort="20000" velocity="2000"/>
-    <joint_properties damping="2.0" friction="2.0"/>
+    <limit effort="11000" velocity="1000"/>
+    <joint_properties damping="1.0" friction="1.0"/>
   </joint>
   <!-- camera joint -->
   <joint type="fixed" name="camera_joint">
-    <origin xyz="0.4 0 0" rpy="0 0 0"/>
+    <origin xyz="0.22 0 0" rpy="0 0 0"/>
     <child link="camera"/>
     <parent link="chassis"/>
@@ -208,5 +211,5 @@
   <!-- laser rangefinder joint -->
   <joint type="fixed" name="hokuyo_joint">
-    <origin xyz="0.30 0 0.2" rpy="0 0 0"/>
+    <origin xyz="0.165 0 0.07" rpy="0 0 0"/>
     <child link="hokuyo"/>
     <parent link="chassis"/>
